File: ESP_DCF77_Emulator.brd (EAGLE design)
At the start: 22 x 26 mm, 18 parts, among them Q1 BC847SMD, Q2 REG1117-33, Q3 ESP01

Commit message: added .gitignore to versioned files Firmware is now in another folder to make the Arduino IDE happy
Parts:
- R1: value 12k -> 100R
- R2: value 10k -> 4k7
Changed lines of the file:
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@@
 <attribute name="VALUE" x="16.905" y="13.175" size="1.27" layer="27" rot="R180"/>
 </element>
-<element name="R1" library="rcl" package="R0603" value="12k" x="23" y="9" smashed="yes" rot="R270">
+<element name="R1" library="rcl" package="R0603" value="100R" x="23" y="9" smashed="yes" rot="R270">
 <attribute name="NAME" x="23.3" y="10.5" size="0.7" layer="25" font="vector" ratio="12" rot="R90"/>
 <attribute name="VALUE" x="21.095" y="9.635" size="1.27" layer="27" rot="R270"/>
@@
 <attribute name="VALUE" x="14.365" y="15.095" size="1.27" layer="27"/>
 </element>
-<element name="R2" library="rcl" package="R0603" value="10k" x="15" y="6.5" smashed="yes" rot="R270">
+<element name="R2" library="rcl" package="R0603" value="4k7" x="15" y="6.5" smashed="yes" rot="R270">
 <attribute name="NAME" x="15.7" y="7" size="0.7" layer="25" font="vector" ratio="12" rot="R270"/>
 <attribute name="VALUE" x="13.095" y="7.135" size="1.27" layer="27" rot="R270"/>
