File: ESP_DCF77_Emulator.sch (EAGLE design)
At the start: 18 parts, among them Q1 BC847SMD, Q2 REG1117-33, Q3 ESP01

Commit message: added .gitignore to versioned files Firmware is now in another folder to make the Arduino IDE happy
Parts:
- R1: value 12k -> 100R
- R2: value 10k -> 4k7
Changed lines of the file:
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@@
 <part name="FRAME1" library="frames" library_urn="urn:adsk.eagle:library:229" deviceset="A4L-LOC" device=""/>
 <part name="Q3" library="esp8266modules" deviceset="ESP01" device=""/>
-<part name="R1" library="rcl" deviceset="R-EU_" device="R0603" value="12k"/>
+<part name="R1" library="rcl" deviceset="R-EU_" device="R0603" value="100R"/>
 <part name="GND3" library="supply1" deviceset="GND" device=""/>
 <part name="GND4" library="supply1" deviceset="GND" device=""/>
@@
 <part name="P+1" library="supply1" deviceset="+5V" device=""/>
 <part name="GND1" library="supply1" deviceset="GND" device=""/>
-<part name="R2" library="rcl" deviceset="R-EU_" device="R0603" value="10k"/>
+<part name="R2" library="rcl" deviceset="R-EU_" device="R0603" value="4k7"/>
 <part name="SJ1" library="jumper" library_urn="urn:adsk.eagle:library:252" deviceset="SJ2W" device="" package3d_urn="urn:adsk.eagle:package:15474/1"/>
 <part name="P+3" library="supply1" deviceset="+5V" device=""/>
